Commit message: Add collision to wheel_link

File: urdf/weed_robot.xacro (robot description, xacro)
@@ -3,5 +3,4 @@
 <xacro:arg name="meshes" default="true"/>
 <xacro:include filename="$(find weed_robot_description)/urdf/material.xacro"/>
-<xacro:include filename="$(find weed_robot_description)/urdf/gazebo.xacro"/>
 <xacro:include filename="$(find weed_robot_description)/urdf/macro.xacro"/>
 <xacro:property name="config_yaml" value="$(find weed_robot_description)/config/weed_robot.yaml"/>
@@ -123,5 +122,4 @@
   <axis xyz="0 0 1"/>
   <limit lower="${-25/180*pi}" upper="${36/180*pi}" effort="1000" velocity="0.01"/>
-  <dynamics damping="1000"/>
 </joint>
 <!-- Fork front-right -->
@@ -164,5 +162,4 @@
   <axis xyz="0 0 1"/>
   <limit lower="${-36/180*pi}" upper="${25/180*pi}" effort="1000" velocity="0.01"/>
-  <dynamics damping="1000"/>
 </joint>
 <!-- Steer -->
@@ -174,5 +171,4 @@
   <axis xyz="0 0 1"/>
   <limit lower="${-30/180*pi}" upper="${30/180*pi}" effort="1000" velocity="0.01"/>
-  <dynamics damping="1000"/>
 </joint>
 <!-- Fork rear-left -->
@@ -437,5 +433,17 @@
 </joint>
 <!-- Wheel -->
-<link name="wheel_link"/>
+<link name="wheel_link">
+  <inertial>
+    <origin xyz="0 0 0" rpy="0 0 0"/>
+    <mass value="${config['wheel']['mass']}"/>
+    <xacro:cylinder_inertia link_config="${config['wheel']}"/>
+  </inertial>
+  <collision>
+    <origin xyz="0 0 0" rpy="1.5708 0 0"/>
+    <geometry>
+      <xacro:cylinder_geometry link_config="${config['wheel']}"/>
+    </geometry>
+  </collision>
+</link>
 <joint name="base_wheel_joint" type="continuous">
   <parent link="base_link"/>

Commit message: Rename dummy and base links to base and chassis

File: urdf/weed_robot.xacro (robot description, xacro)
@@ -6,8 +6,8 @@
 <xacro:property name="config_yaml" value="$(find weed_robot_description)/config/weed_robot.yaml"/>
 <xacro:property name="config" value="${load_yaml(config_yaml)}"/>
-<!-- Dummy -->
-<link name="dummy_link"/>
+<!-- Base -->
+<link name="base_link"/>
 <!-- Chassis -->
-<link name="base_link">
+<link name="chassis_link">
   <inertial>
     <origin xyz="0 0 0" rpy="0 0 0"/>
@@ -34,5 +34,5 @@
   </collision>
 </link>
-<gazebo reference="base_link">
+<gazebo reference="chassis_link">
   <visual>
     <material>
@@ -41,7 +41,8 @@
   </visual>
 </gazebo>
-<joint name="dummy_joint" type="fixed">
-  <parent link="dummy_link"/>
-  <child link="base_link"/>
+<joint name="base_chassis_joint" type="fixed">
+  <parent link="base_link"/>
+  <child link="chassis_link"/>
+  <origin xyz="0 0 0.83" rpy="0 0 0"/>
 </joint>
 <!-- Panels -->
@@ -78,6 +79,6 @@
   </visual>
 </gazebo>
-<joint name="base_panels_joint" type="fixed">
-  <parent link="base_link"/>
+<joint name="chassis_panels_joint" type="fixed">
+  <parent link="chassis_link"/>
   <child link="panels_link"/>
   <origin xyz="0 0 0.1875" rpy="0 0 0"/>
@@ -116,6 +117,6 @@
   </visual>
 </gazebo>
-<joint name="base_fork_fl_joint" type="revolute">
-  <parent link="base_link"/>
+<joint name="chassis_fork_fl_joint" type="revolute">
+  <parent link="chassis_link"/>
   <child link="fork_fl_link"/>
   <origin rpy="0 0 0" xyz="0.791 0.527 -0.292"/>
@@ -156,6 +157,6 @@
   </visual>
 </gazebo>
-<joint name="base_fork_fr_joint" type="revolute">
-  <parent link="base_link"/>
+<joint name="chassis_fork_fr_joint" type="revolute">
+  <parent link="chassis_link"/>
   <child link="fork_fr_link"/>
   <origin xyz="0.791 -0.527 -0.292" rpy="0 0 0"/>
@@ -165,6 +166,6 @@
 <!-- Steer -->
 <link name="steer_link"/>
-<joint name="base_steer_joint" type="revolute">
-  <parent link="base_link"/>
+<joint name="chassis_steer_joint" type="revolute">
+  <parent link="chassis_link"/>
   <child link="steer_link"/>
   <origin xyz="0.791 0 -0.292" rpy="0 0 0"/>
@@ -205,6 +206,6 @@
   </visual>
 </gazebo>
-<joint name="base_fork_rl_joint" type="fixed">
-  <parent link="base_link"/>
+<joint name="chassis_fork_rl_joint" type="fixed">
+  <parent link="chassis_link"/>
   <child link="fork_rl_link"/>
   <origin xyz="-0.791 0.527 -0.292" rpy="0 0 0"/>
@@ -243,6 +244,6 @@
   </visual>
 </gazebo>
-<joint name="base_fork_rr_joint" type="fixed">
-  <parent link="base_link"/>
+<joint name="chassis_fork_rr_joint" type="fixed">
+  <parent link="chassis_link"/>
   <child link="fork_rr_link"/>
   <origin xyz="-0.791 -0.527 -0.292" rpy="0 0 0"/>
@@ -446,6 +447,6 @@
   </collision>
 </link>
-<joint name="base_wheel_joint" type="continuous">
-  <parent link="base_link"/>
+<joint name="chassis_wheel_joint" type="continuous">
+  <parent link="chassis_link"/>
   <child link="wheel_link"/>
   <origin xyz="-0.791 0 -0.558" rpy="0 0 0"/>

Commit message: Rename base_link as base_link_vis to avoid confusion with the base_link used by other nodes

File: urdf/weed_robot.xacro (robot description, xacro)
@@ -7,5 +7,5 @@
 <xacro:property name="config" value="${load_yaml(config_yaml)}"/>
 <!-- Base -->
-<link name="base_link"/>
+<link name="base_link_vis"/>
 <!-- Chassis -->
 <link name="chassis_link">
@@ -42,5 +42,5 @@
 </gazebo>
 <joint name="base_chassis_joint" type="fixed">
-  <parent link="base_link"/>
+  <parent link="base_link_vis"/>
   <child link="chassis_link"/>
   <origin xyz="0 0 0.83" rpy="0 0 0"/>

Commit message: Add sprayers link

File: urdf/weed_robot.xacro (robot description, xacro)
@@ -44,5 +44,5 @@
   <parent link="base_link_vis"/>
   <child link="chassis_link"/>
-  <origin xyz="0 0 0.83" rpy="0 0 0"/>
+  <origin xyz="0.791 0 0.83" rpy="0 0 0"/>
 </joint>
 <!-- Panels -->
@@ -84,4 +84,42 @@
   <origin xyz="0 0 0.1875" rpy="0 0 0"/>
 </joint>
+<!-- Sprayers -->
+<link name="sprayers_link">
+  <inertial>
+    <origin xyz="0 0 0" rpy="0 0 0"/>
+    <mass value="${config['sprayers']['mass']}"/>
+    <xacro:box_inertia link_config="${config['sprayers']}"/>
+  </inertial>
+  <visual>
+    <origin xyz="0 0 0" rpy="0 0 0"/>
+    <geometry>
+      <xacro:if value="$(arg meshes)">
+        <mesh filename="package://weed_robot_description/meshes/sprayers.stl"/>
+      </xacro:if>
+      <xacro:unless value="$(arg meshes)">
+        <xacro:box_geometry link_config="${config['sprayers']}"/>
+      </xacro:unless>
+    </geometry>
+    <material name="dark_grey"/>
+  </visual>
+  <collision>
+    <origin xyz="0 0 0" rpy="0 0 0"/>
+    <geometry>
+      <xacro:box_geometry link_config="${config['sprayers']}"/>
+    </geometry>
+  </collision>
+</link>
+<gazebo reference="sprayers_link">
+  <visual>
+    <material>
+      <xacro:gmaterial color="dark_grey"/>
+    </material>
+  </visual>
+</gazebo>
+<joint name="chassis_sprayers_joint" type="fixed">
+  <parent link="chassis_link"/>
+  <child link="sprayers_link"/>
+  <origin xyz="-1.216 0 -0.080" rpy="0 0 0"/>
+</joint>
 <!-- Fork front-left -->
 <link name="fork_fl_link">
@@ -120,7 +158,8 @@
   <parent link="chassis_link"/>
   <child link="fork_fl_link"/>
-  <origin rpy="0 0 0" xyz="0.791 0.527 -0.292"/>
+  <origin xyz="0.791 0.527 -0.292" rpy="0 0 0"/>
   <axis xyz="0 0 1"/>
-  <limit lower="${-25/180*pi}" upper="${36/180*pi}" effort="1000" velocity="0.01"/>
+  <limit lower="${-28.391/180*pi}" upper="${40.186/180*pi}" effort="1000" velocity="0.01"/> <!-- calculado con radio de giro 2.40m -->
+  <safety_controller soft_lower_limit="${-27.986/180*pi}" soft_upper_limit="${39.443/180*pi}" k_velocity="10" k_position="15"/> <!-- calculado con radio de giro 2.45m -->
 </joint>
 <!-- Fork front-right -->
@@ -162,5 +201,6 @@
   <origin xyz="0.791 -0.527 -0.292" rpy="0 0 0"/>
   <axis xyz="0 0 1"/>
-  <limit lower="${-36/180*pi}" upper="${25/180*pi}" effort="1000" velocity="0.01"/>
+  <limit lower="${-40.186/180*pi}" upper="${28.391/180*pi}" effort="1000" velocity="0.01"/>
+  <safety_controller soft_lower_limit="${-39.443/180*pi}" soft_upper_limit="${27.986/180*pi}" k_velocity="10" k_position="15"/>
 </joint>
 <!-- Steer -->
@@ -171,5 +211,6 @@
   <origin xyz="0.791 0 -0.292" rpy="0 0 0"/>
   <axis xyz="0 0 1"/>
-  <limit lower="${-30/180*pi}" upper="${30/180*pi}" effort="1000" velocity="0.01"/>
+  <limit lower="${-33.392/180*pi}" upper="${33.392/180*pi}" effort="1000" velocity="0.01"/>
+  <safety_controller soft_lower_limit="${-32.851/180*pi}" soft_upper_limit="${32.851/180*pi}" k_velocity="10" k_position="15"/>
 </joint>
 <!-- Fork rear-left -->
@@ -279,8 +320,8 @@
 </link>
 <gazebo reference="wheel_fl_link">
-  <kp value="1000000"/>
-  <kd value="1"/>
-  <mu1 value="10"/>
-  <mu2 value="10"/>
+  <kp value="${config['wheel']['kp']}"/>
+  <kd value="${config['wheel']['kd']}"/>
+  <mu1 value="${config['wheel']['mu1']}"/>
+  <mu2 value="${config['wheel']['mu2']}"/>
   <visual>
     <material>
@@ -325,8 +366,8 @@
 </link>
 <gazebo reference="wheel_fr_link">
-  <kp value="1000000"/>
-  <kd value="1"/>
-  <mu1 value="10"/>
-  <mu2 value="10"/>
+  <kp value="${config['wheel']['kp']}"/>
+  <kd value="${config['wheel']['kd']}"/>
+  <mu1 value="${config['wheel']['mu1']}"/>
+  <mu2 value="${config['wheel']['mu2']}"/>
   <visual>
     <material>
@@ -371,8 +412,8 @@
 </link>
 <gazebo reference="wheel_rl_link">
-  <kp value="1000000"/>
-  <kd value="1"/>
-  <mu1 value="10"/>
-  <mu2 value="10"/>
+  <kp value="${config['wheel']['kp']}"/>
+  <kd value="${config['wheel']['kd']}"/>
+  <mu1 value="${config['wheel']['mu1']}"/>
+  <mu2 value="${config['wheel']['mu2']}"/>
   <visual>
     <material>
@@ -417,8 +458,8 @@
 </link>
 <gazebo reference="wheel_rr_link">
-  <kp value="1000000"/>
-  <kd value="1"/>
-  <mu1 value="10"/>
-  <mu2 value="10"/>
+  <kp value="${config['wheel']['kp']}"/>
+  <kd value="${config['wheel']['kd']}"/>
+  <mu1 value="${config['wheel']['mu1']}"/>
+  <mu2 value="${config['wheel']['mu2']}"/>
   <visual>
     <material>

Commit message: Add texture to solar panels mesh

File: urdf/weed_robot.xacro (robot description, xacro)
@@ -57,5 +57,6 @@
     <geometry>
       <xacro:if value="$(arg meshes)">
-        <mesh filename="package://weed_robot_description/meshes/panels.stl"/>
+        <!-- <mesh filename="package://weed_robot_description/meshes/panels.stl"/> -->
+        <mesh filename="package://weed_robot_description/meshes/panels.dae"/>
       </xacro:if>
       <xacro:unless value="$(arg meshes)">
@@ -72,5 +73,5 @@
   </collision>
 </link>
-<gazebo reference="panels_link">
+<!-- <gazebo reference="panels_link">
   <visual>
     <material>
@@ -78,5 +79,5 @@
     </material>
   </visual>
-</gazebo>
+</gazebo> -->
 <joint name="chassis_panels_joint" type="fixed">
   <parent link="chassis_link"/>
